Commit message: Install worlds dir and add urdf_config.rviz for bringup
Co-Authored-By: Claude Fable 5 <noreply@anthropic.com>

File: agbot_bringup/urdf/agbot_camera.urdf.xacro (robot description, xacro)
@@ -54,5 +54,5 @@
     <parent link="mid_mount"/>
     <child  link="camera_mount_link"/>
-    <origin xyz="-0.10 0 0.10" rpy="0 0 0"/>
+    <origin xyz="-0.1 0 0.10" rpy="0 0 0"/>
   </joint>
   <!-- ─── Camera body ─────────────────────────────────────────── -->

Commit message: Add display.launch.xml, rear camera, and commented front-deck camera origin
- display.launch.xml: RViz-only URDF visualization (no Gazebo) using the
  same JACKAL_URDF_EXTRAS robot_description as agbot_gazebo.launch
- agbot_camera.urdf.xacro: refactor camera body/optical frame/Gazebo
  sensor into an agbot_cam xacro macro (forward camera keeps all
  historical names and /camera/* topics), add rear camera at
  mid_mount xyz=-0.05 0 0.225 yawed 180 deg publishing /camera_rear/*,
  and add commented-out low front-deck origin xyz=0.19 0 0.025 for the
  camera-occlusion relocation test

Co-Authored-By: Claude Fable 5 <noreply@anthropic.com>

File: agbot_bringup/urdf/agbot_camera.urdf.xacro (robot description, xacro)
@@ -2,5 +2,5 @@
 <robot xmlns:xacro="http://www.ros.org/wiki/xacro">
   <!--
-    AgBot forward camera with physical mount stand.
+    AgBot cameras with physical mount stand.
     Included via JACKAL_URDF_EXTRAS into jackal.urdf.xacro.
     Parent link: mid_mount (top-centre of Jackal chassis).
@@ -9,8 +9,10 @@
                            front face flush with x=0, body extends to x=-0.20 m
                            centre at xyz="-0.10  0  0.10"
-      camera_link        — sensor origin at xyz="0  0  0.225"
+      camera_link        — forward sensor origin at xyz="0  0  0.225"
                            (camera bottom = 0.20 m = top of stand)
-      camera_optical_frame — CV convention (z forward, x right, y down)
-                             used as the image header frame_id
+      camera_rear_link   — rear sensor at xyz="-0.05 0 0.225", yawed 180°
+                           (back-to-back with the forward camera on the stand)
+      *_optical_frame    — CV convention (z forward, x right, y down)
+                           used as the image header frame_id
   -->
   <!-- Mount stand dimensions (m) -->
@@ -56,84 +58,102 @@
     <origin xyz="-0.1 0 0.10" rpy="0 0 0"/>
   </joint>
-  <!-- ─── Camera body ─────────────────────────────────────────── -->
-  <link name="camera_link">
-    <visual>
-      <geometry>
-        <box size="${cam_length} ${cam_width} ${cam_height}"/>
-      </geometry>
-      <material name="dark_grey"/>
-    </visual>
-    <collision>
-      <geometry>
-        <box size="${cam_length} ${cam_width} ${cam_height}"/>
-      </geometry>
-    </collision>
-    <inertial>
-      <mass value="0.05"/>
-      <origin xyz="0 0 0" rpy="0 0 0"/>
-      <inertia
-        ixx="${0.05*(cam_width*cam_width   + cam_height*cam_height)/12}"
-        ixy="0" ixz="0"
-        iyy="${0.05*(cam_length*cam_length + cam_height*cam_height)/12}"
-        iyz="0"
-        izz="${0.05*(cam_length*cam_length + cam_width*cam_width)/12}"/>
-    </inertial>
-  </link>
-  <!-- camera centre: x=0, y=0 (robot centre), z=cam_z above mid_mount.
-       Camera bottom (cam_z - cam_height/2 = 0.20 m) sits on stand top. -->
-  <joint name="base_camera_joint" type="fixed">
-    <parent link="mid_mount"/>
-    <child  link="camera_link"/>
-    <origin xyz="0 0 ${cam_z}" rpy="0 0 0"/>
-  </joint>
-  <!-- ─── Optical frame (CV convention) ───────────────────────── -->
-  <!-- z forward, x right, y down.
-       Transform: -90° around X, then -90° around Z. -->
-  <link name="camera_optical_frame"/>
-  <joint name="camera_optical_joint" type="fixed">
-    <parent link="camera_link"/>
-    <child  link="camera_optical_frame"/>
-    <origin xyz="0 0 0" rpy="-1.5707963 0 -1.5707963"/>
-  </joint>
-  <!-- ─── Gazebo sensor and material ──────────────────────────── -->
   <gazebo reference="camera_mount_link">
     <material>Gazebo/DarkGrey</material>
   </gazebo>
-  <gazebo reference="camera_link">
-    <material>Gazebo/DarkGrey</material>
-    <sensor type="camera" name="agbot_camera">
-      <update_rate>30.0</update_rate>
-      <camera name="head">
-        <!-- 80° horizontal FOV — wide enough to see row boundaries -->
-        <horizontal_fov>1.3962634</horizontal_fov>
-        <image>
-          <width>640</width>
-          <height>480</height>
-          <format>R8G8B8</format>
-        </image>
-        <clip>
-          <near>0.02</near>
-          <far>300</far>
-        </clip>
-        <noise>
-          <type>gaussian</type>
-          <mean>0.0</mean>
-          <stddev>0.007</stddev>
-        </noise>
-      </camera>
-      <plugin name="camera_controller" filename="libgazebo_ros_camera.so">
-        <alwaysOn>true</alwaysOn>
-        <updateRate>30.0</updateRate>
-        <cameraName>camera</cameraName>
-        <imageTopicName>image_raw</imageTopicName>
-        <cameraInfoTopicName>camera_info</cameraInfoTopicName>
-        <frameName>camera_optical_frame</frameName>
-        <distortionK1>0.0</distortionK1>
-        <distortionK2>0.0</distortionK2>
-        <distortionK3>0.0</distortionK3>
-        <distortionT1>0.0</distortionT1>
-        <distortionT2>0.0</distortionT2>
-      </plugin>
-    </sensor>
-  </gazebo>
+  <!-- ─── Camera macro: body + optical frame + Gazebo sensor ──── -->
+  <!-- name=camera keeps all historical names/topics of the forward
+       camera (camera_link, base_camera_joint, camera_optical_frame,
+       sensor agbot_camera, plugin camera_controller, /camera/*). -->
+  <xacro:macro name="agbot_cam" params="name xyz rpy">
+    <link name="${name}_link">
+      <visual>
+        <geometry>
+          <box size="${cam_length} ${cam_width} ${cam_height}"/>
+        </geometry>
+        <material name="dark_grey"/>
+      </visual>
+      <collision>
+        <geometry>
+          <box size="${cam_length} ${cam_width} ${cam_height}"/>
+        </geometry>
+      </collision>
+      <inertial>
+        <mass value="0.05"/>
+        <origin xyz="0 0 0" rpy="0 0 0"/>
+        <inertia
+          ixx="${0.05*(cam_width*cam_width   + cam_height*cam_height)/12}"
+          ixy="0" ixz="0"
+          iyy="${0.05*(cam_length*cam_length + cam_height*cam_height)/12}"
+          iyz="0"
+          izz="${0.05*(cam_length*cam_length + cam_width*cam_width)/12}"/>
+      </inertial>
+    </link>
+    <joint name="base_${name}_joint" type="fixed">
+      <parent link="mid_mount"/>
+      <child  link="${name}_link"/>
+      <origin xyz="${xyz}" rpy="${rpy}"/>
+    </joint>
+    <!-- Optical frame, CV convention: z forward, x right, y down.
+         Transform: -90° around X, then -90° around Z (relative to the
+         camera link, so it is identical for front and rear cameras). -->
+    <link name="${name}_optical_frame"/>
+    <joint name="${name}_optical_joint" type="fixed">
+      <parent link="${name}_link"/>
+      <child  link="${name}_optical_frame"/>
+      <origin xyz="0 0 0" rpy="-1.5707963 0 -1.5707963"/>
+    </joint>
+    <gazebo reference="${name}_link">
+      <material>Gazebo/DarkGrey</material>
+      <sensor type="camera" name="agbot_${name}">
+        <update_rate>30.0</update_rate>
+        <camera name="head">
+          <!-- 80° horizontal FOV — wide enough to see row boundaries -->
+          <horizontal_fov>1.3962634</horizontal_fov>
+          <image>
+            <width>640</width>
+            <height>480</height>
+            <format>R8G8B8</format>
+          </image>
+          <clip>
+            <near>0.02</near>
+            <far>300</far>
+          </clip>
+          <noise>
+            <type>gaussian</type>
+            <mean>0.0</mean>
+            <stddev>0.007</stddev>
+          </noise>
+        </camera>
+        <plugin name="${name}_controller" filename="libgazebo_ros_camera.so">
+          <alwaysOn>true</alwaysOn>
+          <updateRate>30.0</updateRate>
+          <cameraName>${name}</cameraName>
+          <imageTopicName>image_raw</imageTopicName>
+          <cameraInfoTopicName>camera_info</cameraInfoTopicName>
+          <frameName>${name}_optical_frame</frameName>
+          <distortionK1>0.0</distortionK1>
+          <distortionK2>0.0</distortionK2>
+          <distortionK3>0.0</distortionK3>
+          <distortionT1>0.0</distortionT1>
+          <distortionT2>0.0</distortionT2>
+        </plugin>
+      </sensor>
+    </gazebo>
+  </xacro:macro>
+  <!-- ─── Forward camera ──────────────────────────────────────── -->
+  <!-- camera centre: x=0, y=0 (robot centre), z=cam_z above mid_mount.
+       Camera bottom (cam_z - cam_height/2 = 0.20 m) sits on stand top. -->
+  <xacro:agbot_cam name="camera" xyz="0 0 ${cam_z}" rpy="0 0 0"/>
+  <!-- Alternative low/front mount (occlusion test): camera on the front
+       deck, lens just behind the +0.210 m front edge of the chassis
+       (parent stays mid_mount). z=0.025 puts the 0.05 m-tall camera
+       body's bottom on the deck plane. To test, comment the line above
+       and uncomment the line below; consider also commenting the stand
+       (camera_mount_link + camera_mount_joint) since it stays behind.
+  <xacro:agbot_cam name="camera" xyz="0.19 0 0.025" rpy="0 0 0"/>
+  -->
+  <!-- ─── Rear camera (blocked-row back-out) ──────────────────── -->
+  <!-- Back-to-back with the forward camera on the stand, yawed 180°.
+       Publishes /camera_rear/image_raw, frame camera_rear_optical_frame. -->
+  <xacro:agbot_cam name="camera_rear" xyz="-0.05 0 ${cam_z}" rpy="0 0 3.14159265"/>
 </robot>

Commit message: Mirror the rear camera onto the rear deck, matching the low front mount
Both cameras now sit at z=0.025 with the same 0.02 m inset from their
respective deck edges: front x=+0.19, rear x=-0.19. The rear camera was
left on the 0.225 m stand when the front one moved down, so the reverse
view no longer matched the forward view.

That match is load-bearing: the back-out steers from the rear camera
reusing the MPC with unchanged signs, which assumes the reverse view is
the geometric twin of the forward view.

The low mount is now the standard; the tall stand line is kept commented
as a record of the original geometry.

Co-Authored-By: Claude Opus 5 <noreply@anthropic.com>

File: agbot_bringup/urdf/agbot_camera.urdf.xacro (robot description, xacro)
@@ -6,11 +6,12 @@
     Parent link: mid_mount (top-centre of Jackal chassis).
     Layout (all offsets relative to mid_mount):
-      camera_mount_link  — 20×5×20 cm stand
-                           front face flush with x=0, body extends to x=-0.20 m
-                           centre at xyz="-0.10  0  0.10"
-      camera_link        — forward sensor origin at xyz="0  0  0.225"
-                           (camera bottom = 0.20 m = top of stand)
-      camera_rear_link   — rear sensor at xyz="-0.05 0 0.225", yawed 180°
-                           (back-to-back with the forward camera on the stand)
+      camera_mount_link  — 20×5×20 cm stand, kept for the TALL mount option
+                           (currently unused; both cameras are deck-mounted)
+      camera_link        — forward sensor on the front deck at
+                           xyz="0.19  0  0.025"
+      camera_rear_link   — rear sensor MIRRORED about the robot centre at
+                           xyz="-0.19  0  0.025", yawed 180°. Same height as
+                           the front camera, same inset from its deck edge, so
+                           the reverse view matches the forward view.
       *_optical_frame    — CV convention (z forward, x right, y down)
                            used as the image header frame_id
@@ -56,5 +57,5 @@
     <parent link="mid_mount"/>
     <child  link="camera_mount_link"/>
-    <origin xyz="-0.1 0 0.10" rpy="0 0 0"/>
+    <origin xyz="-0.025 0 0.10" rpy="0 0 0"/>
   </joint>
   <gazebo reference="camera_mount_link">
@@ -141,19 +142,23 @@
     </gazebo>
   </xacro:macro>
-  <!-- ─── Forward camera ──────────────────────────────────────── -->
-  <!-- camera centre: x=0, y=0 (robot centre), z=cam_z above mid_mount.
-       Camera bottom (cam_z - cam_height/2 = 0.20 m) sits on stand top. -->
-  <xacro:agbot_cam name="camera" xyz="0 0 ${cam_z}" rpy="0 0 0"/>
-  <!-- Alternative low/front mount (occlusion test): camera on the front
-       deck, lens just behind the +0.210 m front edge of the chassis
-       (parent stays mid_mount). z=0.025 puts the 0.05 m-tall camera
-       body's bottom on the deck plane. To test, comment the line above
-       and uncomment the line below; consider also commenting the stand
-       (camera_mount_link + camera_mount_joint) since it stays behind.
+  <!-- ─── Forward camera (LOW deck mount — the standard now) ──── -->
+  <!-- On the front deck, lens just inside the +0.210 m front edge of the
+       chassis (parent stays mid_mount). z=0.025 puts the 0.05 m-tall camera
+       body's bottom on the deck plane. The low mount is preferred over the
+       tall stand: it sees the row boundaries closer in and matches the
+       physical GPU robot. -->
   <xacro:agbot_cam name="camera" xyz="0.19 0 0.025" rpy="0 0 0"/>
-  -->
+  <!-- Tall stand mount, kept as a record of the original geometry. If it is
+       ever re-enabled, move the rear camera back to the stand as well
+       (xyz="-0.05 0 ${cam_z}") so the two stay mirrored. -->
+  <!-- <xacro:agbot_cam name="camera" xyz="0 0 ${cam_z}" rpy="0 0 0"/> -->
   <!-- ─── Rear camera (blocked-row back-out) ──────────────────── -->
-  <!-- Back-to-back with the forward camera on the stand, yawed 180°.
+  <!-- MIRROR of the forward camera about the robot centre: same z, same
+       0.02 m inset from its deck edge, yawed 180°. The back-out steers from
+       this camera reusing the MPC with UNCHANGED signs (image mirror ×
+       reversed motion cancel), which assumes the reverse view is the
+       geometric twin of the forward view — a different height or inset would
+       break that assumption and mistune the reverse leg.
        Publishes /camera_rear/image_raw, frame camera_rear_optical_frame. -->
-  <xacro:agbot_cam name="camera_rear" xyz="-0.05 0 ${cam_z}" rpy="0 0 3.14159265"/>
+  <xacro:agbot_cam name="camera_rear" xyz="-0.19 0 0.025" rpy="0 0 3.14159265"/>
 </robot>

Commit message: Remove the unused camera stand and move the LiDAR forward behind the front camera
Co-Authored-By: Claude Opus 5.5 <noreply@anthropic.com>

File: agbot_bringup/urdf/agbot_camera.urdf.xacro (robot description, xacro)
@@ -2,5 +2,5 @@
 <robot xmlns:xacro="http://www.ros.org/wiki/xacro">
   <!--
-    AgBot cameras with physical mount stand, plus the optional 3D LiDAR.
+    AgBot cameras, plus the optional 3D LiDAR.
     Included via JACKAL_URDF_EXTRAS into jackal.urdf.xacro.
     xacro arg lidar:=true (default false) also includes
@@ -8,6 +8,4 @@
     Parent link: mid_mount (top-centre of Jackal chassis).
     Layout (all offsets relative to mid_mount):
-      camera_mount_link  — 20×5×20 cm stand, kept for the TALL mount option
-                           (currently unused; both cameras are deck-mounted)
       camera_link        — forward sensor on the front deck at
                            xyz="0.19  0  0.025"
@@ -19,49 +17,8 @@
                            used as the image header frame_id
   -->
-  <!-- Mount stand dimensions (m) -->
-  <xacro:property name="mount_length" value="0.05"/>
-  <xacro:property name="mount_width"  value="0.20"/>
-  <xacro:property name="mount_height" value="0.20"/>
   <!-- Camera sensor body dimensions (m) -->
   <xacro:property name="cam_length" value="0.01"/>
   <xacro:property name="cam_width"  value="0.10"/>
   <xacro:property name="cam_height" value="0.05"/>
-  <!-- half-height shortcuts -->
-  <xacro:property name="cam_z" value="0.225"/>  <!-- 0.20 + cam_height/2 -->
-  <!-- ─── Mount stand ─────────────────────────────────────────── -->
-  <link name="camera_mount_link">
-    <visual>
-      <geometry>
-        <box size="${mount_length} ${mount_width} ${mount_height}"/>
-      </geometry>
-      <material name="dark_grey"/>
-    </visual>
-    <collision>
-      <geometry>
-        <box size="${mount_length} ${mount_width} ${mount_height}"/>
-      </geometry>
-    </collision>
-    <inertial>
-      <mass value="0.3"/>
-      <origin xyz="0 0 0" rpy="0 0 0"/>
-      <inertia
-        ixx="${0.3*(mount_width*mount_width   + mount_height*mount_height)/12}"
-        ixy="0" ixz="0"
-        iyy="${0.3*(mount_length*mount_length + mount_height*mount_height)/12}"
-        iyz="0"
-        izz="${0.3*(mount_length*mount_length + mount_width*mount_width)/12}"/>
-    </inertial>
-  </link>
-  <!-- centre of box: x=-0.10 m (front face at x=0, extends behind),
-                      y= 0.00 m (centred),
-                      z= 0.10 m (half of 0.20 m height, rests on platform) -->
-  <joint name="camera_mount_joint" type="fixed">
-    <parent link="mid_mount"/>
-    <child  link="camera_mount_link"/>
-    <origin xyz="-0.025 0 0.10" rpy="0 0 0"/>
-  </joint>
-  <gazebo reference="camera_mount_link">
-    <material>Gazebo/DarkGrey</material>
-  </gazebo>
   <!-- ─── Camera macro: body + optical frame + Gazebo sensor ──── -->
   <!-- name=camera keeps all historical names/topics of the forward
@@ -147,12 +104,9 @@
   <!-- On the front deck, lens just inside the +0.210 m front edge of the
        chassis (parent stays mid_mount). z=0.025 puts the 0.05 m-tall camera
-       body's bottom on the deck plane. The low mount is preferred over the
-       tall stand: it sees the row boundaries closer in and matches the
-       physical GPU robot. -->
+       body's bottom on the deck plane. The low mount sees the row
+       boundaries closer in and matches the physical GPU robot. (The old
+       20 cm camera stand, camera_mount_link, was removed 2026-10-14; it is
+       in git history.) -->
   <xacro:agbot_cam name="camera" xyz="0.19 0 0.025" rpy="0 0 0"/>
-  <!-- Tall stand mount, kept as a record of the original geometry. If it is
-       ever re-enabled, move the rear camera back to the stand as well
-       (xyz="-0.05 0 ${cam_z}") so the two stay mirrored. -->
-  <!-- <xacro:agbot_cam name="camera" xyz="0 0 ${cam_z}" rpy="0 0 0"/> -->
   <!-- ─── Rear camera (blocked-row back-out) ──────────────────── -->
   <!-- MIRROR of the forward camera about the robot centre: same z, same

File: agbot_bringup/urdf/agbot_lidar.urdf.xacro (robot description, xacro)
@@ -5,5 +5,6 @@
     Included by agbot_camera.urdf.xacro only when the xacro arg lidar:=true,
     so the default URDF (and the laptop sim's RTF) is unchanged.
-    Layout (all offsets relative to mid_mount, the deck top centre):
+    Layout (all offsets relative to mid_mount, the deck top centre). The
+    stack sits at x = lidar_mount_x (0.10), just BEHIND the front camera:
       lidar_standoff_link — 7 cm standoff on the deck
       lidar_housing_link  — 15 cm cube on the standoff, deck +0.07 to +0.22 m
@@ -15,7 +16,10 @@
     carries the same base_link -> velodyne numbers, and a pytest keeps them
     equal.
-    Clearance: the lowest VLP-16 beam (-15 deg) from 0.258 m reaches deck
-    height (0) about 0.96 m out, so it clears the front camera (x=0.19,
-    z<=0.05) and the deck edge.
+    Clearance: the camera is 0.09 m in front of the scan centre, where the
+    lowest VLP-16 beam (-15 deg, from 0.258 m) is still 0.23 m up — far
+    above the 0.05 m camera body; that beam reaches deck height only ~0.96 m
+    out, past the deck edge. The housing is behind the camera, so it is not
+    in the camera's view, and well forward of the rear camera (x=-0.19,
+    facing backwards).
     The vertical LiDAR (/ns2) is not modelled — it is not used for SLAM.
     ⚠ The Gazebo plugin needs ros-noetic-velodyne-gazebo-plugins.
@@ -26,5 +30,8 @@
   <xacro:property name="lidar_standoff_width"  value="0.10"/>
   <xacro:property name="lidar_housing_size"    value="0.15"/>
-  <xacro:property name="lidar_mount_x"         value="0.0"/>
+  <!-- Housing centre, forward of mid_mount. 0.10 puts the housing's front
+       face (0.10 + 0.075 = 0.175) 1 cm behind the front camera body, which
+       spans x = 0.185-0.195. Moved forward from 0.0 on 2026-10-14. -->
+  <xacro:property name="lidar_mount_x"         value="0.10"/>
   <!-- Must match the frame_id the robot's driver stamps on
        /ns1/velodyne_points (LIDAR_notes.md). -->
